File: boards/v2_512k_flash/vectrex-cartridge-512k.kicad_pcb (KiCad board)
At the start: 2 copper layers, 54 x 66 mm, 18 parts, among them CON1 vectrex-edge-connector, U1 SST39SF040 (PLCC-32 socket), U2 74HC377, U3 74HC00, U4 74HC1G32

Commit message: 512K board: routed with a router of our own - straight bus lanes, 0/45/90 degree tracks
The PLCC socket turned and moved up so the address bus reaches it from inside; the latch's
unused inputs D4-D8 tied to GND; unused fingers (/HALT, /NMI, /IRQ) without copper. DRC with
the project's rules: no unconnected items, no clearance errors. New renders, copper layers,
schematic and Gerbers; routing/ holds the router and its plan (route.py removed).

Co-Authored-By: Claude Opus 5.5 <noreply@anthropic.com>
Parts:
- moved R1 19.3 mm to (161.0, 89.0)
- moved U1 10.3 mm to (146.8, 99.7), turned to -90 degrees
- turned U2 to 180 degrees
Connections:
- U2 pad 13: C_D4 -> GND
- U2 pad 14: C_D5 -> GND
- U2 pad 17: C_D6 -> GND
- U2 pad 18: C_D7 -> GND
- U2 pad 8: C_D3 -> GND
Routing:
- net GND: track 174.3 -> 47.6 mm, vias 4 -> 9
- net C_A13: track 35.7 -> 140.1 mm, vias 0 -> 5
- net C_D6: track 99.6 -> 27.3 mm, vias 4 -> 0
- net C_D0: track 116.3 -> 46.4 mm, vias 2 -> 1
- net C_D1: track 101.1 -> 39.8 mm, vias 5 -> 2
- net C_D7: track 73.9 -> 27.1 mm, vias 0 -> 2
- net BA18: track 64.8 -> 19.7 mm, vias 3 -> 0
- net V-PB6: track 48.7 -> 92.2 mm, vias 0 -> 3
- net C_D5: track 68.5 -> 32.4 mm, vias 3 -> 0
- net C_A8: track 63.1 -> 27.9 mm, vias 4 -> 0
- net C_A14: track 59.3 -> 93.6 mm, vias 2 -> 6
- net C_A11: track 57.6 -> 26.8 mm, vias 2 -> 0
- net C_A10: track 54.9 -> 25.8 mm, vias 2 -> 0
- net C_D4: track 59.5 -> 32.1 mm, vias 2 -> 1
- net C_A12: track 25.1 -> 51.5 mm
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